File: MM_PowerBoard_Draft/MM_PowerBoard_Draft.kicad_pcb (KiCad board)
At the start: 2 copper layers, 80 x 60 mm, 51 parts, among them IC1 74HC14D, IC2 TPS61023DRLR, J1 JST_Battery, J2 2x16_Motherboard, Q2 AO3400A, U1 CH224K, U2 TPS22810DRV, U3 TB6612FNG, U4 AP2112K-3.3, U5 TPS22810DRV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

Commit message: Few violations left
Parts:
- removed TP1: TestPoint_2Pole, TestPoint:TestPoint_Bridge_Pitch2.54mm_Drill1.0mm
Routing:
- net /Out: track 22.9 -> 129.1 mm, vias 2 -> 8
- net /Sense_-: track 0.35 -> 76.5 mm, vias 0 -> 2
- net /5V: track 3.11 -> 74.9 mm, vias 0 -> 2
- net /MOTOR2_CTRL1: track 0.00 -> 51.6 mm, vias 0 -> 3
- net /Sense_+: track 0.00 -> 50.9 mm, vias 0 -> 2
- net /MOTOR2_A_OUT: track 50.4 -> 4.18 mm, vias 1 -> 0
- net /HV: track 0.00 -> 43.7 mm, vias 0 -> 1
- net /3V3: track 18.1 -> 58.4 mm, vias 2 -> 1
- net /EXT_LOAD2_OUT: track 9.04 -> 48.7 mm, vias 0 -> 2
- net /EXT_LOAD1_OUT: track 13.0 -> 49.3 mm, vias 0 -> 1
- net /CTRL_EXT_LOAD1: track 0.00 -> 34.5 mm, vias 0 -> 1
- net /FAST_CHARGE_CTRL: track 0.00 -> 32.4 mm, vias 0 -> 1
- net /MOTOR3_A_OUT: track 0.00 -> 29.0 mm, vias 0 -> 1
- net /I2C1_SDA: track 0.00 -> 25.8 mm, vias 0 -> 1
- net /MOTOR3_CTRL1: track 0.00 -> 24.7 mm, vias 0 -> 1
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- removed copper zone on F.Cu, net /Out
