File: MM_PowerBoard_Draft/MM_PowerBoard_Draft.kicad_pcb (KiCad board)
At the start: 2 copper layers, 80 x 60 mm, 50 parts, among them IC1 74HC14D, IC2 TPS61023DRLR, J1 JST_Battery, J2 2x16_Motherboard, Q2 AO3400A, U1 CH224K, U2 TPS22810DRV, U3 TB6612FNG, U4 AP2112K-3.3, U5 TPS22810DRV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

Commit message: Latest
Parts:
- removed R10, R7: 10, Custom-Footprints:R0603
- added JP1: SolderJumper_2_Open, Jumper:SolderJumper-2_P1.3mm_Open_Pad1.0x1.5mm, F.Cu at (136.5, 77.5)
- C12, C8: value 1e-6 -> 10e-6
- Q2: footprint Package_TO_SOT_SMD:SOT-23 -> Custom-Footprints:SOT-23-3_L2.9-W1.3-P1.90-LS2.4-BR
- U4: footprint Package_TO_SOT_SMD:SOT-23-5 -> Custom-Footprints:SOT-25-5_L2.9-W1.6-P0.95-LS2.8-BL
Routing:
- net /MOTOR2_A_OUT: track 4.18 -> 153.1 mm, vias 0 -> 1
- net /MOTOR2_B_OUT: track 3.00 -> 78.0 mm
- net /HV: track 43.7 -> 69.1 mm, vias 1 -> 3
- net /Out: track 129.1 -> 153.1 mm, vias 8 -> 14
- net /EXT_LOAD1_OUT: track 49.3 -> 67.8 mm
- net /CHARGER_OUT: track 22.8 -> 41.1 mm
- net GND: track 72.8 -> 85.9 mm, vias 41 -> 40
- net /MOTOR1_CTRL1: track 5.44 -> 18.0 mm, vias 0 -> 2
- net Net-(U1-CFG1): track 0.00 -> 9.68 mm, vias 0 -> 2
- net /VBUS: track 25.2 -> 31.6 mm
- net /3V3: track 58.4 -> 61.7 mm, vias 1 -> 3
- net Net-(U4-EN): track 6.24 -> 3.06 mm
- net /MOTOR1_CTRL2: track 11.7 -> 14.0 mm
- net Net-(Q2-D): track 6.45 -> 4.51 mm
- net Net-(U1-VBUS): track 4.17 -> 5.90 mm
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