File: MM_PowerBoard_Draft/MM_PowerBoard_Draft.kicad_sch (KiCad schematic)
At the start: 40 parts, among them IC1 74HC14D, J1 JST_Battery, J2 2x16_Motherboard, J3 USB_C_Receptacle, Q1 PMOS, Q2 AO3400A, SW1 SW_SPDT, U1 CYPD3177-24LQ, U2 TPS22810DRV, U3 TB6612FNG, U4 AP2112K-3.3, U5 TPS22810DRV, U6 TB6612FNG, U7 INA219AxDCN, U8 BQ24074RGT, U9 TPS613222ADBZ

Commit message: PCB in progress.
Parts:
- removed J3: USB_C_Receptacle, symbol Connector:USB_C_Receptacle
- removed Q1: PMOS, symbol Simulation_SPICE:PMOS
- removed SW1: SW_SPDT, symbol Switch:SW_SPDT
- removed U1: CYPD3177-24LQ, Package_DFN_QFN:QFN-24-1EP_4x4mm_P0.5mm_EP2.75x2.75mm, symbol Interface_USB:CYPD3177-24LQ
- removed U9: TPS613222ADBZ, Package_TO_SOT_SMD:SOT-23, symbol Regulator_Switching:TPS613222ADBZ
- added C13: 22uF, Custom-Footprints:C1206, symbol Device:C
- added C14: 1e-6, Custom-Footprints:C0603, symbol Device:C
- added C15, C16: 10e-6, Custom-Footprints:C0603, symbol Device:C
- added IC2: TPS61023DRLR, Custom-Footprints:SOT-563_L1.6-W1.2-P0.50-LS1.6-BR, symbol TPS61023DRLR:TPS61023DRLR
- added JP1: SolderJumper_2_Open, Jumper:SolderJumper-2_P1.3mm_Open_Pad1.0x1.5mm, symbol Jumper:SolderJumper_2_Open
- added R11: 100, Custom-Footprints:R0603, symbol Device:R_US
- added R12: 750k, Custom-Footprints:R0603, symbol Device:R_US
- added R13: 100k, Custom-Footprints:R1206, symbol Device:R_US
- added R14, R16: 10k, Custom-Footprints:R0603, symbol Device:R_US
- added R15: 6.8k, Custom-Footprints:R0603, symbol Device:R_US
- added R17: 1.1k, Custom-Footprints:R0603, symbol Device:R_US
- added U1: CH224K, Custom-Footprints:ESSOP-10_L4.9-W3.9-P1.0-LS6.0-TL-EP, symbol Custom-Symbols:CH224K
- added U9: SS-12D10-G050, Custom-Footprints:SW-TH_SS-12D10-G050, symbol Custom-Symbols:SS-12D10-G050
- added USBC1: TYPE-C-31-M-12, Custom-Footprints:USB-C_SMD-TYPE-C-31-M-12, symbol Custom-Symbols:TYPE-C-31-M-12
- C1, C10, C2, C3, C4, C5, C6, C7: footprint Capacitor_SMD:C_0805_2012Metric -> Custom-Footprints:C0603
- C11: value 2200e-12 -> 1e-6; footprint Capacitor_SMD:C_0805_2012Metric -> Custom-Footprints:C0603
- C12, C8: value 1e-7 -> 1e-6; footprint Capacitor_SMD:C_0805_2012Metric -> Custom-Footprints:C0603
- C9: value 2200e-9 -> 1e-6; footprint Capacitor_SMD:C_0805_2012Metric -> Custom-Footprints:C0603
- IC1: footprint Package_SO:SOIC-14_3.9x8.7mm_P1.27mm -> Custom-Footprints:SOIC-14_L8.7-W3.9-P1.27-LS6.0-BL
- L1: value L -> 1uH; footprint Inductor_SMD:L_0805_2012Metric -> Inductor_SMD:L_Sunlord_SWPA4030S
- R1, R10, R2, R3, R4, R5, R6, R7, R8, R9: footprint Resistor_SMD:R_0603_1608Metric -> Custom-Footprints:R0603
- R20: renamed from R1(0.1Ohm)1; value PE2512FKE7W0R1L -> 0.1Ω; footprint Current_Sense:RESC6432X89N -> Custom-Footprints:R2512
- U8: footprint Package_DFN_QFN:VQFN-16-1EP_3x3mm_P0.5mm_EP1.6x1.6mm -> Custom-Footprints:VQFN-16_L3.0-W3.0-P0.50-TL-EP1.7
Connections:
- net BATTERY is gone; now on net Sense_-: J2.14 (Pin_14)
- net Motor4_A_Out is gone; now on net EXT_LOAD1_OUT: J2.21 (Pin_21)
- net 5V: now also C13.1, IC2.6 (VOUT), R12.1
- net FAST_CHARGE_CTRL: now also R11.1; no longer Q2.1 (G)
- net GND: now also C13.2, C14.2, C15.2, C16.2, IC2.4 (GND), R13.2, R15.1, U1.11 (GND), USBC1.0 (SH), USBC1.1 (SH), USBC1.2 (SH), USBC1.3 (SH), USBC1.A1 (GND), USBC1.A12 (GND), USBC1.B1 (GND), USBC1.B12 (GND)
- net HV: now also JP1.2 (B)
- net Out: now also U3.13 (VM2), U3.14 (VM3), U3.24 (VM1), U6.13 (VM2), U6.14 (VM3), U6.24 (VM1), C15.1, C16.1, IC2.2 (EN), IC2.3 (VIN), R14.2, U9.2; no longer L1.2, U4.3 (EN), U8.10 (OUT), U8.11 (OUT)
- net Sense_-: now also J1.1 (Pin_1)
- removed net BAT_POS: J1.1 (Pin_1), R20.1, U3.13 (VM2), U3.14 (VM3), U3.24 (VM1), U6.13 (VM2), U6.14 (VM3), U6.24 (VM1), U7.1 (IN+)
- net SYS_BAT renamed Sense_+
- net Sense_+: now also R20.1, U7.1 (IN+); no longer C6.1
- new net: IC2.1 (FB), R12.2, R13.1
- new net: IC2.5 (SW), L1.2
- new net: Q2.1 (G), R11.2
- new net: R14.1, U4.3 (EN)
- new net: R15.2, U1.9 (CFG1)
- new net: C14.1, R17.2, U1.1 (VDD)
- new net: U1.4 (DP), U1.5 (DM)
- new net: R16.2, U1.8 (VBUS)
- new net CC1: U1.7 (CC1), USBC1.A5 (CC1)
- new net CC2: U1.6 (CC2), USBC1.B5 (CC2)
- new net CHARGER_OUT: C6.1, U8.10 (OUT), U8.11 (OUT), U9.3
- new net VBUS: JP1.1 (A), R16.1, R17.1, USBC1.A4 (VBUS), USBC1.A9 (VBUS), USBC1.B4 (VBUS), USBC1.B9 (VBUS)
- no-connect marks 1 -> 18
Other:
- moved on the sheet: C11, C2

Commit message: Latest
Parts:
- removed R10, R7: 10, Custom-Footprints:R0603, symbol Device:R_US
- C12, C8: value 1e-6 -> 10e-6
- Q2: footprint Package_TO_SOT_SMD:SOT-23 -> Custom-Footprints:SOT-23-3_L2.9-W1.3-P1.90-LS2.4-BR
- U4: footprint Package_TO_SOT_SMD:SOT-23-5 -> Custom-Footprints:SOT-25-5_L2.9-W1.6-P0.95-LS2.8-BL
